File: Pedal/Pedal/Pedal.kicad_sch (KiCad schematic)
At the start: 22 parts, among them J1 Conn_01x02, J2 Conn_01x02, U1 YAAJ_BluePill_Part_Like, U2 MCP2561-E-SN, U3 AP63200WU

Commit message: lista la placa para imprimir
Connections:
- net +3.3V: now also U1.20 (3V3)
- net CAN_RXD: now also U1.16 (PB8); no longer U1.36 (PB11)
- net CAN_TXD: now also U1.17 (PB9); no longer U1.35 (PB10)
- net GND: now also U1.39 (GND), U1.40 (GND)
Other:
- moved on the sheet: U1

Commit message: listorti
Parts:
- added C10: 1uF, Capacitor_SMD:C_0805_2012Metric_Pad1.18x1.45mm_HandSolder, symbol Device:C
Connections:
- net +5V: now also C10.2
- net GND: now also C7.2, C8.2, C10.1
- net at C6.2, R5.1, R6.2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: no longer C7.2, C8.2
Changed lines of the file:
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@@
 	(rectangle
 		(start 193.04 26.67)
-		(end 279.4 104.14)
+		(end 279.4 107.95)
 		(stroke
 			(width 0)
@@
 	)
 	(junction
+		(at 196.85 87.63)
+		(diameter 0)
+		(color 0 0 0 0)
+	)
+	(junction
 		(at 156.21 49.53)
 		(diameter 0)
@@
 	)
 	(junction
+		(at 149.86 59.69)
+		(diameter 0)
+		(color 0 0 0 0)
+	)
+	(junction
 		(at 62.23 49.53)
 		(diameter 0)
@@
 	)
 	(junction
-		(at 143.51 59.69)
-		(diameter 0)
-		(color 0 0 0 0)
-	)
-	(junction
 		(at 71.12 49.53)
 		(diameter 0)
@@
 	)
 	(junction
+		(at 215.9 99.06)
+		(diameter 0)
+		(color 0 0 0 0)
+	)
+	(junction
 		(at 93.98 138.43)
 		(diameter 0)
@@
 	(wire
 		(pts
+			(xy 149.86 59.69) (xy 156.21 59.69)
+		)
+		(stroke
+			(width 0)
+			(type default)
+		)
+	)
+	(wire
+		(pts
 			(xy 60.96 127) (xy 60.96 128.27)
 		)
@@
 	(wire
 		(pts
-			(xy 143.51 59.69) (xy 156.21 59.69)
+			(xy 215.9 99.06) (xy 215.9 90.17)
+		)
+		(stroke
+			(width 0)
+			(type default)
+		)
+	)
+	(wire
+		(pts
+			(xy 143.51 59.69) (xy 149.86 59.69)
 		)
 		(stroke
@@
 	(wire
 		(pts
+			(xy 196.85 87.63) (xy 196.85 91.44)
+		)
+		(stroke
+			(width 0)
+			(type default)
+		)
+	)
+	(wire
+		(pts
 			(xy 156.21 49.53) (xy 143.51 49.53)
 		)
@@
 	(wire
 		(pts
+			(xy 196.85 99.06) (xy 215.9 99.06)
+		)
+		(stroke
+			(width 0)
+			(type default)
+		)
+	)
+	(wire
+		(pts
 			(xy 73.66 137.16) (xy 73.66 129.54)
 		)
@@
 	(wire
 		(pts
-			(xy 132.08 59.69) (xy 143.51 59.69)
-		)
-		(stroke
-			(width 0)
-			(type default)
-		)
-	)
-	(wire
-		(pts
 			(xy 49.53 49.53) (xy 49.53 53.34)
 		)
@@
 	(wire
 		(pts
+			(xy 149.86 59.69) (xy 149.86 68.58)
+		)
+		(stroke
+			(width 0)
+			(type default)
+		)
+	)
+	(wire
+		(pts
 			(xy 143.51 49.53) (xy 143.51 50.8)
 		)
@@
 	(wire
 		(pts
-			(xy 215.9 97.79) (xy 215.9 90.17)
+			(xy 215.9 101.6) (xy 215.9 99.06)
 		)
 		(stroke
@@
 	(symbol
 		(lib_id "power:GND")
+		(at 149.86 68.58 0)
+		(unit 1)
+		(exclude_from_sim no)
+		(in_bom yes)
+		(on_board yes)
+		(dnp no)
+		(fields_autoplaced yes)
+		(property "Reference" "#PWR018"
+			(at 149.86 74.93 0)
+			(effects
+				(font
+					(size 1.27 1.27)
+				)
+				(hide yes)
+			)
+		)
+		(property "Value" "GND"
+			(at 149.86 73.66 0)
+			(effects
+				(font
+					(size 1.27 1.27)
+				)
+			)
+		)
+		(property "Footprint" ""
+			(at 149.86 68.58 0)
+			(effects
+				(font
+					(size 1.27 1.27)
+				)
+				(hide yes)
+			)
+		)
+		(property "Datasheet" ""
+			(at 149.86 68.58 0)
+			(effects
+				(font
+					(size 1.27 1.27)
+				)
+				(hide yes)
+			)
+		)
+		(property "Description" "Power symbol creates a global label with name \"GND\" , ground"
+			(at 149.86 68.58 0)
+			(effects
+				(font
+					(size 1.27 1.27)
+				)
+				(hide yes)
+			)
+		)
+		(pin "1"
+		)
+		(instances
+			(project "Pedal"
+				(path "/74379d8d-28c5-49b9-b3e9-1f584bef7bb9"
+					(reference "#PWR018")
+					(unit 1)
+				)
+			)
+		)
+	)
+	(symbol
+		(lib_id "power:GND")
 		(at 275.59 46.99 0)
 		(unit 1)
@@
 	(symbol
 		(lib_id "Device:C")
+		(at 196.85 95.25 180)
+		(unit 1)
+		(exclude_from_sim no)
+		(in_bom yes)
+		(on_board yes)
+		(dnp no)
+		(fields_autoplaced yes)
+		(property "Reference" "C10"
+			(at 200.66 93.9799 0)
+			(effects
+				(font
+					(size 1.27 1.27)
+				)
+				(justify right)
+			)
+		)
+		(property "Value" "1uF"
+			(at 200.66 96.5199 0)
+			(effects
+				(font
+					(size 1.27 1.27)
+				)
+				(justify right)
+			)
+		)
+		(property "Footprint" "Capacitor_SMD:C_0805_2012Metric_Pad1.18x1.45mm_HandSolder"
+			(at 195.8848 91.44 0)
+			(effects
+				(font
+					(size 1.27 1.27)
+				)
+				(hide yes)
+			)
+		)
+		(property "Datasheet" "~"
+			(at 196.85 95.25 0)
+			(effects
+				(font
+					(size 1.27 1.27)
+				)
+				(hide yes)
+			)
+		)
+		(property "Description" "Unpolarized capacitor"
+			(at 196.85 95.25 0)
+			(effects
+				(font
+					(size 1.27 1.27)
+				)
+				(hide yes)
+			)
+		)
+		(pin "2"
+		)
+		(pin "1"
+		)
+		(instances
+			(project "Pedal"
+				(path "/74379d8d-28c5-49b9-b3e9-1f584bef7bb9"
+					(reference "C10")
+					(unit 1)
+				)
+			)
+		)
+	)
+	(symbol
+		(lib_id "Device:C")
 		(at 54.61 127 90)
 		(unit 1)
@@
 	(symbol
 		(lib_id "power:GND")
-		(at 215.9 97.79 0)
+		(at 215.9 101.6 0)
 		(mirror y)
 		(unit 1)
@@
 		(dnp no)
 		(property "Reference" "#PWR016"
-			(at 215.9 104.14 0)
+			(at 215.9 107.95 0)
 			(effects
 				(font
@@
 		)
 		(property "Value" "GND"
-			(at 215.9 102.87 0)
+			(at 215.9 106.68 0)
 			(effects
 				(font
@@
 		)
 		(property "Footprint" ""
-			(at 215.9 97.79 0)
+			(at 215.9 101.6 0)
 			(effects
 				(font
@@
 		)
 		(property "Datasheet" ""
-			(at 215.9 97.79 0)
+			(at 215.9 101.6 0)
 			(effects
 				(font
@@
 		)
 		(property "Description" "Power symbol creates a global label with name \"GND\" , ground"
-			(at 215.9 97.79 0)
-			(effects
-				(font
+			(at 215.9 101.6 0)
+			(effects
+				(font
