File: Pedal/Pedal/Pedal.kicad_pcb (KiCad board)
At the start: 2 copper layers, 50 x 66.5 mm, 24 parts, among them J1 Conn_01x02, J2 Conn_01x02, U1 YAAJ_BluePill_Part_Like, U2 MCP2561-E-SN, U3 AP63200WU

Commit message: lista la placa para imprimir
Parts:
- added G***: LOGO, LOGO, B.Cu at (62.0, 77.2)
- C1, C2, C3, C4, C5, C6, C7, C8, C9, L1, R2, R3, R4, R5, R6, R7, U2, U3: moved to B.Cu
- moved REF** 65.3 mm to (62.0, 36.5)
- moved REF** 53.5 mm to (62.0, 91.0), turned to 180 degrees
- moved RV1 43.4 mm to (60.5, 53.2), turned to 0 degrees
- moved J2 36.5 mm to (102.5, 86.8), turned to 180 degrees
- moved C8 33.7 mm to (102.0, 76.0)
- moved U3 33.2 mm to (95.8, 80.2), turned to 180 degrees
- moved R6 33.0 mm to (104.5, 76.0), turned to -90 degrees
- moved L1 31.2 mm to (94.3, 70.0), turned to 0 degrees
- moved C3 30.0 mm to (93.5, 84.2), turned to 0 degrees
- moved R3 29.2 mm to (76.2, 40.8), turned to 180 degrees
- moved C7 28.2 mm to (99.5, 76.0)
- moved C4 26.7 mm to (93.5, 86.5), turned to 0 degrees
- moved R7 26.7 mm to (103.8, 70.8), turned to -90 degrees
- moved C6 26.6 mm to (94.3, 76.0)
- moved R5 25.4 mm to (97.0, 76.0)
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Connections:
- U1 pad 16: unconnected-(U1-PB8-Pad16) -> CAN_RXD
- U1 pad 17: unconnected-(U1-PB9-Pad17) -> CAN_TXD
- U1 pad 39: unconnected-(U1-GND-Pad39) -> GND
- U1 pad 40: unconnected-(U1-GND-Pad40) -> GND
Routing:
- net +5V: track 46.7 -> 94.1 mm
- net GND: track 126.7 -> 157.1 mm
- net Net-(J1-Pin_1): track 11.1 -> 40.9 mm
- net Net-(J1-Pin_2): track 21.9 -> 51.1 mm
- net +3.3V: track 42.8 -> 17.4 mm
- net Net-(U3-FB): track 36.6 -> 12.6 mm
- net Net-(U2-SPLIT): track 4.39 -> 27.5 mm
- net POT_VALUE: track 42.4 -> 26.7 mm
- net CAN_TXD: track 0.00 -> 12.4 mm
- net +24V: track 22.2 -> 11.3 mm
- net Net-(C1-Pad2): track 16.1 -> 6.75 mm
- net CAN_RXD: track 0.00 -> 7.56 mm
- net Net-(U3-SW): track 11.2 -> 16.1 mm
- net Net-(U3-BST): track 2.97 -> 3.59 mm
Other:
- board text added: "LGBS 2025"

Commit message: listorti
Parts:
- added C10: 1uF, Capacitor_SMD:C_0805_2012Metric_Pad1.18x1.45mm_HandSolder, B.Cu at (85.0, 57.0)
- moved G*** 36.5 mm to (79.0, 45.0)
- moved R3 18.5 mm to (94.5, 43.5), turned to 0 degrees
- moved R4 16.4 mm to (94.5, 46.5), turned to 180 degrees
- moved R2 14.0 mm to (93.5, 49.8), turned to -90 degrees
- moved C8 13.9 mm to (95.0, 64.0), turned to 0 degrees
- moved C1 11.0 mm to (90.2, 46.5), turned to 0 degrees
- moved C9 11.0 mm to (64.0, 59.2)
- moved R7 10.8 mm to (104.0, 81.5), turned to 90 degrees
- moved C7 10.5 mm to (95.0, 66.5), turned to 0 degrees
- moved C2 6.44 mm to (95.0, 61.5)
- moved C6 6.23 mm to (100.5, 76.2)
- moved REF** 6.00 mm to (62.0, 85.0)
- moved R5 5.98 mm to (103.0, 76.2)
- moved R6 5.85 mm to (100.5, 80.2), turned to 180 degrees
- moved L1 4.50 mm to (94.2, 74.5)
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Connections:
- C7 pad 2: Net-(U3-FB) -> GND
- C8 pad 2: Net-(U3-FB) -> GND
Routing:
- net +5V: track 94.1 -> 34.5 mm, vias 0 -> 2
- net Net-(U2-SPLIT): track 27.5 -> 3.09 mm
- net Net-(J1-Pin_1): track 40.9 -> 21.8 mm
- net GND: track 157.1 -> 151.6 mm
- net Net-(U3-SW): track 16.1 -> 11.4 mm
- net +3.3V: track 17.4 -> 14.6 mm
- net Net-(U3-FB): track 12.6 -> 9.92 mm
- net Net-(J1-Pin_2): track 51.1 -> 49.3 mm
- net Net-(U3-BST): track 3.59 -> 2.37 mm
- net CAN_TXD: track 12.4 -> 13.6 mm
- net Net-(R6-Pad1): track 3.57 -> 2.60 mm
- net Net-(C1-Pad2): track 6.75 -> 7.50 mm
- added copper zone on B.Cu, net GND
Other:
- board size 50 x 66.5 mm -> 50 x 61.5 mm

Commit message: stm arreglada
Parts:
- moved C10 14.7 mm to (84.4, 42.3)
- moved C1 1.69 mm to (91.4, 45.3), turned to -90 degrees
Routing:
- net GND: track 151.6 -> 84.9 mm
- net +3.3V: track 14.6 -> 36.2 mm
- net +5V: track 34.5 -> 45.7 mm
- net POT_VALUE: track 26.7 -> 36.9 mm
- net CAN_RXD: track 7.47 -> 13.9 mm
- net CAN_TXD: track 13.6 -> 17.8 mm
- net unconnected-(U1-PA6-Pad31): track 0.00 -> 0.92 mm
- net unconnected-(U1-PB5-Pad13): track 0.00 -> 0.59 mm
- net unconnected-(U1-PB6-Pad14): track 0.00 -> 0.55 mm
